File: hello.t1616.echo.thruhole.sch (KiCad schematic (older format))
At the start: 4 parts, among them J1 Conn_01x03_Male, J2 Conn_FTDI_01x06_Male, U1 ATtiny1616-S

Commit message: Added thruhole version
Parts:
- J1: footprint fab:Header_SMD_01x03_P2.54mm_Horizontal_Male -> Connector_PinHeader_2.54mm:PinHeader_1x03_P2.54mm_Horizontal
- J2: footprint fab:Header_SMD_01x06_P2.54mm_Horizontal_Male -> Connector_PinHeader_2.54mm:PinHeader_1x06_P2.54mm_Horizontal
Changed lines of the file:
@@
 F 0 "J2" H 7181 3519 50  0000 R CNN
 F 1 "Conn_FTDI_01x06_Male" H 7181 3610 50  0000 R CNN
-F 2 "fab:Header_SMD_01x06_P2.54mm_Horizontal_Male" H 7350 3600 50  0001 C CNN
+F 2 "Connector_PinHeader_2.54mm:PinHeader_1x06_P2.54mm_Horizontal" H 7350 3600 50  0001 C CNN
 F 3 "~" H 7350 3600 50  0001 C CNN
 	1    7350 3600
@@
 F 0 "J1" H 5708 2431 50  0000 C CNN
 F 1 "Conn_01x03_Male" H 5708 2340 50  0000 C CNN
-F 2 "fab:Header_SMD_01x03_P2.54mm_Horizontal_Male" H 5600 2150 50  0001 C CNN
+F 2 "Connector_PinHeader_2.54mm:PinHeader_1x03_P2.54mm_Horizontal" H 5600 2150 50  0001 C CNN
 F 3 "~" H 5600 2150 50  0001 C CNN
 	1    5600 2150
